Commit message: update
- train v2 (optimized)
- data compare v1 vs v2
- test stability v12
--> ready to do vision-based method

File: data/balance_robot.urdf (robot description, URDF)
Before this commit: robot balance_robot_2floor, 8 links, 7 joints
Joints:
- joint base_to_rod_front_left: type fixed -> continuous
- joint base_to_top: type fixed -> continuous
