Commit message: fixed urdf + test ppo

File: hardware/balance_robot.urdf (robot description, URDF)
Before this commit: robot balance_robot_2floor, 8 links, 7 joints
Joints:
- joint base_to_top: type fixed -> continous

Commit message: fix urdf

File: hardware/balance_robot.urdf (robot description, URDF)
Before this commit: robot balance_robot_2floor, 8 links, 7 joints
Joints:
- joint base_to_top: type continous -> fixed

Commit message: fix urdf

File: hardware/balance_robot.urdf (robot description, URDF)
Before this commit: robot balance_robot_2floor, 8 links, 7 joints
Joints:
- joint base_to_left_wheel: origin xyz=0 0.09 -0.04 -> xyz=0 0.09 -0.035
- joint base_to_right_wheel: origin xyz=0 -0.09 -0.04 -> xyz=0 -0.09 -0.035
- joint base_to_rod_back_left: type fixed -> continuous
- joint base_to_rod_back_right: type fixed -> continuous
- joint base_to_rod_front_left: type fixed -> continuous
- joint base_to_rod_front_right: type fixed -> continuous
- joint base_to_top: type fixed -> continuous

Commit message: fix urdf + add in pitch in env2

File: hardware/balance_robot.urdf (robot description, URDF)
Before this commit: robot balance_robot_2floor, 8 links, 7 joints
Joints:
- joint base_to_right_wheel: axis 0 1 0 -> 0 -1 0
- joint base_to_rod_back_left: type continuous -> fixed
- joint base_to_rod_back_right: type continuous -> fixed
- joint base_to_rod_front_left: type continuous -> fixed
- joint base_to_rod_front_right: type continuous -> fixed
- joint base_to_top: origin xyz=0 0 0.05 rpy=0 0 -1.5708 -> xyz=0 0 0.05; type continuous -> fixed

Commit message: update

File: hardware/balance_robot.urdf (robot description, URDF)
Before this commit: robot balance_robot_2floor, 8 links, 7 joints
Joints:
- joint base_to_rod_back_left: type fixed -> continuous
- joint base_to_rod_back_right: type fixed -> continuous
- joint base_to_rod_front_left: type fixed -> continuous
- joint base_to_rod_front_right: type fixed -> continuous
- joint base_to_top: origin xyz=0 0 0.05 -> xyz=0 0 0.05 rpy=0 0 -1.5708; type fixed -> continuous

Commit message: UPDATE BALANCE ROBOT

File: hardware/balance_robot.urdf (robot description, URDF)
Before this commit: robot balance_robot_2floor_stable, 9 links, 8 joints
Links:
- removed link battery
Joints:
- removed joint top_to_battery

Commit message: update

File: hardware/balance_robot.urdf (robot description, URDF)
Before this commit: robot balance_robot_2floor_stable, 8 links, 7 joints
Links:
- added link battery, mass 0.314; collision box size=0.12 0.06 0.02; visual box size=0.12 0.06 0.02
- link base_link: mass 0.25 -> 0.341
- link left_wheel: mass 0.0765 -> 0.049
- link right_wheel: mass 0.0765 -> 0.049
- link rod_back_left: mass 0.01 -> 0.008
- link rod_back_right: mass 0.01 -> 0.008
- link rod_front_left: mass 0.01 -> 0.008
- link rod_front_right: mass 0.01 -> 0.008
- link top_plate: mass 0.20 -> 0.05
Joints:
- added joint top_to_battery: type fixed, parent top_plate, child battery, origin xyz=0 0 0.012 rpy=0 0 0
- joint base_to_left_wheel: origin xyz=0 0.05 -0.035 -> xyz=0 0.05 0
- joint base_to_right_wheel: origin xyz=0 -0.05 -0.035 -> xyz=0 -0.05 0
- joint base_to_rod_back_left: origin xyz=0 0 0 rpy=0 0 -1.5708 -> xyz=-0.06 0.025 0.013 rpy=0 0 0
- joint base_to_rod_back_right: origin xyz=0 0 0 rpy=0 0 -1.5708 -> xyz=-0.06 -0.025 0.013 rpy=0 0 0
- joint base_to_rod_front_left: origin xyz=0 0 0 rpy=0 0 -1.5708 -> xyz=0.06 0.025 0.013 rpy=0 0 0
- joint base_to_rod_front_right: origin xyz=0 0 0 rpy=0 0 -1.5708 -> xyz=0.06 -0.025 0.013 rpy=0 0 0
- joint base_to_top: origin xyz=0 0 0.034 rpy=0 0 -1.5708 -> xyz=0 0 0.034 rpy=0 0 0

Commit message: Update

File: hardware/balance_robot.urdf (robot description, URDF)
Before this commit: robot balance_robot_2floor_stable, 9 links, 8 joints
Joints:
- joint base_to_left_wheel: origin xyz=0 0.05 0 -> xyz=0 0.05 -0.04
- joint base_to_right_wheel: origin xyz=0 -0.05 0 -> xyz=0 -0.05 -0.04

Commit message: update

File: hardware/balance_robot.urdf (robot description, URDF)
Before this commit: robot balance_robot_2floor_stable, 9 links, 8 joints
Links:
- link battery: mass 0.314 -> 0.337; geometry collision box size=0.06 0.03 0.004; visual box size=0.06 0.03 0.004
- link rod_back_left: geometry collision cylinder length=0.05 radius=0.005; visual cylinder length=0.05 radius=0.005
- link rod_back_right: geometry collision cylinder length=0.05 radius=0.005; visual cylinder length=0.05 radius=0.005
- link rod_front_left: geometry collision cylinder length=0.05 radius=0.005; visual cylinder length=0.05 radius=0.005
- link rod_front_right: geometry collision cylinder length=0.05 radius=0.005; visual cylinder length=0.05 radius=0.005
Joints:
- removed joint top_to_battery
- added joint top_plate_to_battery: type fixed, parent top_plate, child battery, origin xyz=0 0 0 rpy=0 0 0
- joint base_to_left_wheel: origin xyz=0 0.05 -0.04 -> xyz=0 0.09 -0.035
- joint base_to_right_wheel: axis 0 1 0 -> 0 -1 0; origin xyz=0 -0.05 -0.04 -> xyz=0 -0.09 -0.035
- joint base_to_rod_back_left: origin xyz=-0.06 0.025 0.013 rpy=0 0 0 -> xyz=0 0 0 rpy=0 0 -1.5708; type fixed -> continuous
- joint base_to_rod_back_right: origin xyz=-0.06 -0.025 0.013 rpy=0 0 0 -> xyz=0 0 0 rpy=0 0 -1.5708; type fixed -> continuous
- joint base_to_rod_front_left: origin xyz=0.06 0.025 0.013 rpy=0 0 0 -> xyz=0 0 0 rpy=0 0 -1.5708; type fixed -> continuous
- joint base_to_rod_front_right: origin xyz=0.06 -0.025 0.013 rpy=0 0 0 -> xyz=0 0 0 rpy=0 0 -1.5708; type fixed -> continuous
- joint base_to_top: origin xyz=0 0 0.034 rpy=0 0 0 -> xyz=0 0 0.05 rpy=0 0 -1.5708; type fixed -> continuous

Commit message: update robot

File: hardware/balance_robot.urdf (robot description, URDF)
Before this commit: robot balance_robot_2floor, 9 links, 8 joints
Joints:
- joint base_to_right_wheel: axis 0 -1 0 -> 0 1 0
- joint base_to_rod_back_left: type continuous -> fixed
- joint base_to_rod_back_right: type continuous -> fixed
- joint base_to_rod_front_left: type continuous -> fixed
- joint base_to_rod_front_right: type continuous -> fixed
- joint base_to_top: type continuous -> fixed

Commit message: update mass + battery

File: hardware/balance_robot.urdf (robot description, URDF)
Before this commit: robot balance_robot_2floor, 8 links, 7 joints
Links:
- added link battery, mass 0.337; collision box size=0.06 0.03 0.004; visual box size=0.06 0.03 0.004
- link base_link: mass 0.279 -> 0.341
- link left_wheel: mass 0.0765 -> 0.049
- link right_wheel: mass 0.0765 -> 0.049
- link rod_back_left: mass None -> 0.008
- link rod_back_right: mass None -> 0.008
- link rod_front_left: mass None -> 0.008
- link rod_front_right: mass None -> 0.008
Joints:
- added joint top_plate_to_battery: type fixed, parent top_plate, child battery, origin xyz=0 0 0 rpy=0 0 0
- joint base_to_left_wheel: origin xyz=0 0.09 -0.04 -> xyz=0 0.09 -0.035
- joint base_to_right_wheel: origin xyz=0 -0.09 -0.04 -> xyz=0 -0.09 -0.035
